Commit message: chore: 更新xacro、ros2_control以支持gazebo

File: src/aubo_moveit_config/config/aubo_i10.ros2_control.xacro (robot description, xacro)
@@ -1,55 +1,60 @@
 <?xml version="1.0"?>
 <robot xmlns:xacro="http://www.ros.org/wiki/xacro">
-  <xacro:macro name="aubo_i10_ros2_control" params="name initial_positions_file">
-    <xacro:property name="initial_positions" value="${load_yaml(initial_positions_file)['initial_positions']}"/>
-    <ros2_control name="${name}" type="system">
-      <hardware>
-        <!-- By default, set up controllers for simulation. This won't work on real hardware -->
-        <!-- <plugin>mock_components/GenericSystem</plugin> -->
-        <plugin>ign_ros2_control/IgnitionSystem</plugin>
-      </hardware>
-      <joint name="shoulder_joint">
-        <command_interface name="position"/>
-        <state_interface name="position">
-          <param name="initial_value">${initial_positions['shoulder_joint']}</param>
-        </state_interface>
-        <state_interface name="velocity"/>
-      </joint>
-      <joint name="upperArm_joint">
-        <command_interface name="position"/>
-        <state_interface name="position">
-          <param name="initial_value">${initial_positions['upperArm_joint']}</param>
-        </state_interface>
-        <state_interface name="velocity"/>
-      </joint>
-      <joint name="foreArm_joint">
-        <command_interface name="position"/>
-        <state_interface name="position">
-          <param name="initial_value">${initial_positions['foreArm_joint']}</param>
-        </state_interface>
-        <state_interface name="velocity"/>
-      </joint>
-      <joint name="wrist1_joint">
-        <command_interface name="position"/>
-        <state_interface name="position">
-          <param name="initial_value">${initial_positions['wrist1_joint']}</param>
-        </state_interface>
-        <state_interface name="velocity"/>
-      </joint>
-      <joint name="wrist2_joint">
-        <command_interface name="position"/>
-        <state_interface name="position">
-          <param name="initial_value">${initial_positions['wrist2_joint']}</param>
-        </state_interface>
-        <state_interface name="velocity"/>
-      </joint>
-      <joint name="wrist3_joint">
-        <command_interface name="position"/>
-        <state_interface name="position">
-          <param name="initial_value">${initial_positions['wrist3_joint']}</param>
-        </state_interface>
-        <state_interface name="velocity"/>
-      </joint>
-    </ros2_control>
-  </xacro:macro>
+    <xacro:macro name="aubo_i10_ros2_control" params="name initial_positions_file">
+        <xacro:property name="initial_positions" value="${load_yaml(initial_positions_file)['initial_positions']}"/>
+        <gazebo>
+            <plugin filename="ign_ros2_control-system" name="ign_ros2_control::IgnitionROS2ControlPlugin">
+                <parameters>/home/xvshuo/work/scl/gazebo_moviet2/src/aubo_moveit_config/config/ros2_controllers.yaml</parameters>
+            </plugin>
+        </gazebo>
+        <ros2_control name="${name}" type="system">
+            <hardware>
+                <!-- By default, set up controllers for simulation. This won't work on real hardware -->
+                <!-- <plugin>mock_components/GenericSystem</plugin> -->
+                <plugin>ign_ros2_control/IgnitionSystem</plugin>
+            </hardware>
+            <joint name="shoulder_joint">
+                <command_interface name="position"/>
+                <state_interface name="position">
+                    <param name="initial_value">${initial_positions['shoulder_joint']}</param>
+                </state_interface>
+                <state_interface name="velocity"/>
+            </joint>
+            <joint name="upperArm_joint">
+                <command_interface name="position"/>
+                <state_interface name="position">
+                    <param name="initial_value">${initial_positions['upperArm_joint']}</param>
+                </state_interface>
+                <state_interface name="velocity"/>
+            </joint>
+            <joint name="foreArm_joint">
+                <command_interface name="position"/>
+                <state_interface name="position">
+                    <param name="initial_value">${initial_positions['foreArm_joint']}</param>
+                </state_interface>
+                <state_interface name="velocity"/>
+            </joint>
+            <joint name="wrist1_joint">
+                <command_interface name="position"/>
+                <state_interface name="position">
+                    <param name="initial_value">${initial_positions['wrist1_joint']}</param>
+                </state_interface>
+                <state_interface name="velocity"/>
+            </joint>
+            <joint name="wrist2_joint">
+                <command_interface name="position"/>
+                <state_interface name="position">
+                    <param name="initial_value">${initial_positions['wrist2_joint']}</param>
+                </state_interface>
+                <state_interface name="velocity"/>
+            </joint>
+            <joint name="wrist3_joint">
+                <command_interface name="position"/>
+                <state_interface name="position">
+                    <param name="initial_value">${initial_positions['wrist3_joint']}</param>
+                </state_interface>
+                <state_interface name="velocity"/>
+            </joint>
+        </ros2_control>
+    </xacro:macro>
 </robot>

File: src/aubo_moveit_config/config/aubo_i10.urdf.xacro (robot description, xacro)
@@ -1,9 +1,9 @@
 <?xml version="1.0"?>
 <robot xmlns:xacro="http://www.ros.org/wiki/xacro" name="aubo_i10">
-    <xacro:arg name="initial_positions_file" default="initial_positions.yaml" />
+    <xacro:arg name="initial_positions_file" default="$(find aubo_moveit_config)/config/initial_positions.yaml" />
     <!-- Import aubo_i10 urdf file -->
     <xacro:include filename="$(find aubo_description)/urdf/aubo_i10.urdf" />
     <!-- Import control_xacro -->
-    <xacro:include filename="aubo_i10.ros2_control.xacro" />
+    <xacro:include filename="$(find aubo_moveit_config)/config/aubo_i10.ros2_control.xacro" />
     <xacro:aubo_i10_ros2_control name="aubo" initial_positions_file="$(arg initial_positions_file)"/>
 </robot>
