Commit message: 生成新的assistance，用标定工具进行标定

File: src/aubo_description/urdf/aubo_i10.urdf (robot description, URDF)
Before this commit: robot aubo_i10, 8 links, 7 joints
Links:
- added link camera_link, mass 0.1; collision box size=0.05 0.05 0.1; visual box size=0.05 0.05 0.1
Joints:
- added joint camera_joint: type fixed, parent wrist3_Link, child camera_link, origin xyz=0 0 0.06 rpy=0 0 0

Commit message: chore: 更新aubo_description中的文件路径为相对路径

File: src/aubo_description/urdf/aubo_i10.urdf (robot description, URDF)
Before this commit: robot aubo_i10, 9 links, 8 joints
Links:
- link base_link: geometry collision mesh filename=package://aubo_description/meshes/aubo_i10/collision/link0.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; visual mesh filename=package://aubo_description/meshes/aubo_i10/visual/link0.DAE
- link foreArm_Link: geometry collision mesh filename=package://aubo_description/meshes/aubo_i10/collision/link3.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; visual mesh filename=package://aubo_description/meshes/aubo_i10/visual/link3.DAE
- link shoulder_Link: geometry collision mesh filename=package://aubo_description/meshes/aubo_i10/collision/link1.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; visual mesh filename=package://aubo_description/meshes/aubo_i10/visual/link1.DAE
- link upperArm_Link: geometry collision mesh filename=package://aubo_description/meshes/aubo_i10/collision/link2.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; visual mesh filename=package://aubo_description/meshes/aubo_i10/visual/link2.DAE
- link wrist1_Link: geometry collision mesh filename=package://aubo_description/meshes/aubo_i10/collision/link4.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; visual mesh filename=package://aubo_description/meshes/aubo_i10/visual/link4.DAE
- link wrist2_Link: geometry collision mesh filename=package://aubo_description/meshes/aubo_i10/collision/link5.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; visual mesh filename=package://aubo_description/meshes/aubo_i10/visual/link5.DAE
- link wrist3_Link: geometry collision mesh filename=package://aubo_description/meshes/aubo_i10/collision/link6.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; visual mesh filename=package://aubo_description/meshes/aubo_i10/visual/link6.DAE

File: src/aubo_description/urdf/aubo_i10.urdf.xacro (robot description, xacro)
@@ -13,14 +13,14 @@
       <origin xyz="0 0 0" rpy="0 0 0" />
       <geometry>
-        <mesh filename="file:///home/xvshuo/work/scl/auborobot/install/share/aubo_description/meshes/aubo_i10/visual/link0.DAE" />
-      </geometry>
-      <material name="">
-        <color rgba="1 1 1 1" />
-      </material>
-    </visual>
-    <collision>
-      <origin xyz="0 0 0" rpy="0 0 0" />
-      <geometry>
-        <mesh filename="file:///home/xvshuo/work/scl/auborobot/install/share/aubo_description/meshes/aubo_i10/collision/link0.STL" />
+        <mesh filename="package://aubo_description/meshes/aubo_i10/visual/link0.DAE" />
+      </geometry>
+      <material name="">
+        <color rgba="1 1 1 1" />
+      </material>
+    </visual>
+    <collision>
+      <origin xyz="0 0 0" rpy="0 0 0" />
+      <geometry>
+        <mesh filename="package://aubo_description/meshes/aubo_i10/collision/link0.STL" />
       </geometry>
     </collision>
@@ -35,5 +35,5 @@
       <origin xyz="0 0 0" rpy="0 0 0" />
       <geometry>
-        <mesh filename="file:///home/xvshuo/work/scl/auborobot/install/share/aubo_description/meshes/aubo_i10/visual/link1.DAE" />
+        <mesh filename="package://aubo_description/meshes/aubo_i10/visual/link1.DAE" />
       </geometry>
       <material name="">
@@ -44,5 +44,5 @@
       <origin xyz="0 0 0" rpy="0 0 0" />
       <geometry>
-        <mesh filename="file:///home/xvshuo/work/scl/auborobot/install/share/aubo_description/meshes/aubo_i10/collision/link1.STL" />
+        <mesh filename="package://aubo_description/meshes/aubo_i10/collision/link1.STL" />
       </geometry>
     </collision>
@@ -64,5 +64,5 @@
       <origin xyz="0 0 0" rpy="0 0 0" />
       <geometry>
-        <mesh filename="file:///home/xvshuo/work/scl/auborobot/install/share/aubo_description/meshes/aubo_i10/visual/link2.DAE" />
+        <mesh filename="package://aubo_description/meshes/aubo_i10/visual/link2.DAE" />
       </geometry>
       <material name="">
@@ -73,5 +73,5 @@
       <origin xyz="0 0 0" rpy="0 0 0" />
       <geometry>
-        <mesh filename="file:///home/xvshuo/work/scl/auborobot/install/share/aubo_description/meshes/aubo_i10/collision/link2.STL" />
+        <mesh filename="package://aubo_description/meshes/aubo_i10/collision/link2.STL" />
       </geometry>
     </collision>
@@ -93,14 +93,14 @@
       <origin xyz="0 0 0" rpy="0 0 0" />
       <geometry>
-        <mesh filename="file:///home/xvshuo/work/scl/auborobot/install/share/aubo_description/meshes/aubo_i10/visual/link3.DAE" />
-      </geometry>
-      <material name="">
-        <color rgba="1 1 1 1" />
-      </material>
-    </visual>
-    <collision>
-      <origin xyz="0 0 0" rpy="0 0 0" />
-      <geometry>
-        <mesh filename="file:///home/xvshuo/work/scl/auborobot/install/share/aubo_description/meshes/aubo_i10/collision/link3.STL" />
+        <mesh filename="package://aubo_description/meshes/aubo_i10/visual/link3.DAE" />
+      </geometry>
+      <material name="">
+        <color rgba="1 1 1 1" />
+      </material>
+    </visual>
+    <collision>
+      <origin xyz="0 0 0" rpy="0 0 0" />
+      <geometry>
+        <mesh filename="package://aubo_description/meshes/aubo_i10/collision/link3.STL" />
       </geometry>
     </collision>
@@ -122,14 +122,14 @@
       <origin xyz="0 0 0" rpy="0 0 0" />
       <geometry>
-        <mesh filename="file:///home/xvshuo/work/scl/auborobot/install/share/aubo_description/meshes/aubo_i10/visual/link4.DAE" />
-      </geometry>
-      <material name="">
-        <color rgba="1 1 1 1" />
-      </material>
-    </visual>
-    <collision>
-      <origin xyz="0 0 0" rpy="0 0 0" />
-      <geometry>
-        <mesh filename="file:///home/xvshuo/work/scl/auborobot/install/share/aubo_description/meshes/aubo_i10/collision/link4.STL" />
+        <mesh filename="package://aubo_description/meshes/aubo_i10/visual/link4.DAE" />
+      </geometry>
+      <material name="">
+        <color rgba="1 1 1 1" />
+      </material>
+    </visual>
+    <collision>
+      <origin xyz="0 0 0" rpy="0 0 0" />
+      <geometry>
+        <mesh filename="package://aubo_description/meshes/aubo_i10/collision/link4.STL" />
       </geometry>
     </collision>
@@ -151,14 +151,14 @@
       <origin xyz="0 0 0" rpy="0 0 0" />
       <geometry>
-        <mesh filename="file:///home/xvshuo/work/scl/auborobot/install/share/aubo_description/meshes/aubo_i10/visual/link5.DAE" />
-      </geometry>
-      <material name="">
-        <color rgba="1 1 1 1" />
-      </material>
-    </visual>
-    <collision>
-      <origin xyz="0 0 0" rpy="0 0 0" />
-      <geometry>
-        <mesh filename="file:///home/xvshuo/work/scl/auborobot/install/share/aubo_description/meshes/aubo_i10/collision/link5.STL" />
+        <mesh filename="package://aubo_description/meshes/aubo_i10/visual/link5.DAE" />
+      </geometry>
+      <material name="">
+        <color rgba="1 1 1 1" />
+      </material>
+    </visual>
+    <collision>
+      <origin xyz="0 0 0" rpy="0 0 0" />
+      <geometry>
+        <mesh filename="package://aubo_description/meshes/aubo_i10/collision/link5.STL" />
       </geometry>
     </collision>
@@ -180,14 +180,14 @@
       <origin xyz="0 0 0" rpy="0 0 0" />
       <geometry>
-        <mesh filename="file:///home/xvshuo/work/scl/auborobot/install/share/aubo_description/meshes/aubo_i10/visual/link6.DAE" />
-      </geometry>
-      <material name="">
-        <color rgba="1 1 1 1" />
-      </material>
-    </visual>
-    <collision>
-      <origin xyz="0 0 0" rpy="0 0 0" />
-      <geometry>
-        <mesh filename="file:///home/xvshuo/work/scl/auborobot/install/share/aubo_description/meshes/aubo_i10/collision/link6.STL" />
+        <mesh filename="package://aubo_description/meshes/aubo_i10/visual/link6.DAE" />
+      </geometry>
+      <material name="">
+        <color rgba="1 1 1 1" />
+      </material>
+    </visual>
+    <collision>
+      <origin xyz="0 0 0" rpy="0 0 0" />
+      <geometry>
+        <mesh filename="package://aubo_description/meshes/aubo_i10/collision/link6.STL" />
       </geometry>
     </collision>
@@ -206,3 +206,61 @@
     <origin xyz="0.0 0.0 0.0" rpy="0.0 0.0 0.0" />
   </joint>
+  <link name="camera_link">
+    <inertial>
+      <origin xyz="0 0 0" rpy="0 0 0" />
+      <mass value="0.1" />
+      <inertia ixx="0.0001" ixy="0" ixz="0" iyy="0.0001" iyz="0" izz="0.0001" />
+    </inertial>
+    <visual>
+      <origin xyz="0 0 0" rpy="0 0 0" />
+      <geometry>
+        <box size="0.05 0.05 0.1" />
+      </geometry>
+      <material name="black">
+        <color rgba="0 0 0 1" />
+      </material>
+    </visual>
+    <collision>
+      <origin xyz="0 0 0" rpy="0 0 0" />
+      <geometry>
+        <box size="0.05 0.05 0.1" />
+      </geometry>
+    </collision>
+  </link>
+  <joint name="camera_joint" type="fixed">
+    <parent link="wrist3_Link" />
+    <child link="camera_link" />
+    <origin xyz="0 0 0.06" rpy="0 0 0" />
+  </joint>
+  <!-- 定义相机传感器 -->
+  <gazebo reference="camera_link">
+    <sensor type="camera" name="camera">
+      <pose>0 0 0.05 -1.5708 -1.5708 0</pose>
+      <camera>
+        <horizontal_fov>1.047</horizontal_fov>
+        <image>
+          <width>800</width>
+          <height>600</height>
+        </image>
+        <clip>
+          <near>0.1</near>
+          <far>100</far>
+        </clip>
+      </camera>
+      <alwaysOn>true</alwaysOn>
+      <updateRate>15</updateRate>
+      <visualize>true</visualize>
+      <topic>/camera</topic>
+    </sensor>
+  </gazebo>
+  <gazebo>
+    <!-- 相机插件 -->
+    <plugin filename="ignition-gazebo-sensors-system" name="gz::sim::systems::Sensors">
+      <render_engine>ogre</render_engine>
+    </plugin>
+    <!-- ROS2控制插件 -->
+    <plugin name="ign_ros2_control::IgnitionROS2ControlPlugin" filename="ign_ros2_control-system">
+      <parameters>$(find moveit_assistant)/config/ros2_controllers.yaml</parameters>
+    </plugin>
+  </gazebo>
 </robot>

Commit message: chore: 更新相机话题和静态变换
更新了相机话题和静态变换，将左相机和右相机的话题名称分别修改为"/left/camera"和"/right/camera"，并更新了对应的静态变换文件。

File: src/aubo_description/urdf/aubo_i10.urdf (robot description, URDF)
Before this commit: robot aubo_i10, 9 links, 8 joints
Links:
- removed link camera_link
- added link left_camera_link, mass 0.1; collision box size=0.05 0.05 0.1; visual box size=0.05 0.05 0.1
- added link right_camera_link, mass 0.1; collision box size=0.05 0.05 0.1; visual box size=0.05 0.05 0.1
Joints:
- removed joint camera_joint
- added joint left_camera_joint: type fixed, parent wrist3_Link, child left_camera_link, origin xyz=-0.1 0 0.06 rpy=0 0 0
- added joint right_camera_joint: type fixed, parent wrist3_Link, child right_camera_link, origin xyz=0.1 0 0.06 rpy=0 0 0
